File: pcb/K9QW_ATTiny_CW_Keyer/K9QW_ATTiny_CW_Keyer.kicad_sch (KiCad schematic)
At the start: 40 parts, among them J1 Power Input, J2 AudioJack4, J3 AudioJack4, J4 Mounting Hole, Q1 AO3401A, Q2 MMBT2222A, Q3 MMBT3904, Q4 MMBT3904, SW1 Power Switch, SW2 Command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

Commit message: Recommend omitting sidetone LED by default
Parts:
- D3, Q4, R10, R8: now not fitted
- R6: value 220R -> 470R
- R9: value 220R -> 470R; now not fitted
Other:
- note added: "R10 is recommended by buzzer datasheet, but does not appear to make much difference at sidetone frequencies. Omit to save a little power, pad provided to potentially help with any distortion or other issues."
Changed lines of the file:
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@@
 		)
 	)
+	(text "R10 is recommended by buzzer datasheet, but does not \nappear to make much difference at sidetone frequencies.\nOmit to save a little power, pad provided to \npotentially help with any distortion or other issues."
+		(exclude_from_sim no)
+		(at 256.286 60.706 0)
+		(effects
+			(font
+				(size 1.27 1.27)
+			)
+		)
+	)
 	(text "Optional RC-LPF (~1kHz) to filter squarewave \nbefore driving an external audio circuit.\nCut JP4 if LPF is populated.  \nDo no populate LPF and do not cut JP4 if \ndriving a simple piezo disc speaker."
 		(exclude_from_sim no)
@@
 		(in_bom yes)
 		(on_board yes)
-		(dnp no)
+		(dnp yes)
 		(fields_autoplaced yes)
 		(property "Reference" "D3"
@@
 			)
 		)
-		(property "Value" "220R"
+		(property "Value" "470R"
 			(at 190.5 120.6499 0)
 			(effects
@@
 		(in_bom yes)
 		(on_board yes)
-		(dnp no)
+		(dnp yes)
 		(fields_autoplaced yes)
 		(property "Reference" "R8"
@@
 		(in_bom yes)
 		(on_board yes)
-		(dnp no)
+		(dnp yes)
 		(fields_autoplaced yes)
 		(property "Reference" "R10"
@@
 		(in_bom yes)
 		(on_board yes)
-		(dnp no)
+		(dnp yes)
 		(fields_autoplaced yes)
 		(property "Reference" "Q4"
@@
 		(in_bom yes)
 		(on_board yes)
-		(dnp no)
+		(dnp yes)
 		(fields_autoplaced yes)
 		(property "Reference" "R9"
@@
 			)
 		)
-		(property "Value" "220R"
+		(property "Value" "470R"
 			(at 241.3 120.6499 0)
 			(effects
